File: ByteExplore_DevBoard_W_loader/bytexplore_devboard.sch (EAGLE design)
At the start: 91 parts, among them IC1 LM1117MPX-3.3, IC2 STM32F107RCT, IC3 CP2102, IC4 MIC5219, IC6 STM32F103C8T, J1 POWER_JACKPTH, Y1 SMD-CRYSTAL-8MHZ-20PF-20PPM(2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

Commit message: initial commit
Parts:
- C13, C22: value (none) -> 20pf
- C23, C24: value (none) -> 100nf
- R10, R20: value 220 -> 4k7
- R21: value 220 -> 100
- R23: value 220 -> 10k
- R24: value 220 -> 22
- R25: value 220 -> 222
- R26: value 220 -> 100k
- R27: value 220 -> 1k5
- R8, R9: value 220 -> 100K
Changed lines of the file:
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@@
 <part name="C16" library="rcl" library_urn="urn:adsk.eagle:library:334" deviceset="C-EU" device="C0603" package3d_urn="urn:adsk.eagle:package:23616/2" value="10uf"/>
 <part name="IC6" library="micro-stm_v2" deviceset="STM32F103C*T" device="" technology="8"/>
-<part name="C13" library="rcl" library_urn="urn:adsk.eagle:library:334" deviceset="C-EU" device="C0603" package3d_urn="urn:adsk.eagle:package:23616/2"/>
-<part name="C22" library="rcl" library_urn="urn:adsk.eagle:library:334" deviceset="C-EU" device="C0603" package3d_urn="urn:adsk.eagle:package:23616/2"/>
+<part name="C13" library="rcl" library_urn="urn:adsk.eagle:library:334" deviceset="C-EU" device="C0603" package3d_urn="urn:adsk.eagle:package:23616/2" value="20pf"/>
+<part name="C22" library="rcl" library_urn="urn:adsk.eagle:library:334" deviceset="C-EU" device="C0603" package3d_urn="urn:adsk.eagle:package:23616/2" value="20pf"/>
 <part name="GND11" library="supply1" library_urn="urn:adsk.eagle:library:371" deviceset="GND" device=""/>
-<part name="C23" library="rcl" library_urn="urn:adsk.eagle:library:334" deviceset="C-EU" device="C0603" package3d_urn="urn:adsk.eagle:package:23616/2"/>
+<part name="C23" library="rcl" library_urn="urn:adsk.eagle:library:334" deviceset="C-EU" device="C0603" package3d_urn="urn:adsk.eagle:package:23616/2" value="100nf"/>
 <part name="GND19" library="supply1" library_urn="urn:adsk.eagle:library:371" deviceset="GND" device=""/>
 <part name="+3V7" library="supply1" library_urn="urn:adsk.eagle:library:371" deviceset="+3V3" device=""/>
 <part name="+3V8" library="supply1" library_urn="urn:adsk.eagle:library:371" deviceset="+3V3" device=""/>
 <part name="GND20" library="supply1" library_urn="urn:adsk.eagle:library:371" deviceset="GND" device=""/>
-<part name="C24" library="rcl" library_urn="urn:adsk.eagle:library:334" deviceset="C-EU" device="C0603" package3d_urn="urn:adsk.eagle:package:23616/2"/>
-<part name="R8" library="rcl" library_urn="urn:adsk.eagle:library:334" deviceset="R-US_" device="R0603" package3d_urn="urn:adsk.eagle:package:23555/2" value="220"/>
+<part name="C24" library="rcl" library_urn="urn:adsk.eagle:library:334" deviceset="C-EU" device="C0603" package3d_urn="urn:adsk.eagle:package:23616/2" value="100nf"/>
+<part name="R8" library="rcl" library_urn="urn:adsk.eagle:library:334" deviceset="R-US_" device="R0603" package3d_urn="urn:adsk.eagle:package:23555/2" value="100K"/>
 <part name="+3V9" library="supply1" library_urn="urn:adsk.eagle:library:371" deviceset="+3V3" device=""/>
 <part name="GND21" library="supply1" library_urn="urn:adsk.eagle:library:371" deviceset="GND" device=""/>
-<part name="R9" library="rcl" library_urn="urn:adsk.eagle:library:334" deviceset="R-US_" device="R0603" package3d_urn="urn:adsk.eagle:package:23555/2" value="220"/>
+<part name="R9" library="rcl" library_urn="urn:adsk.eagle:library:334" deviceset="R-US_" device="R0603" package3d_urn="urn:adsk.eagle:package:23555/2" value="100K"/>
 <part name="GND22" library="supply1" library_urn="urn:adsk.eagle:library:371" deviceset="GND" device=""/>
 <part name="GND23" library="supply1" library_urn="urn:adsk.eagle:library:371" deviceset="GND" device=""/>
-<part name="R10" library="rcl" library_urn="urn:adsk.eagle:library:334" deviceset="R-US_" device="R0603" package3d_urn="urn:adsk.eagle:package:23555/2" value="220"/>
-<part name="R20" library="rcl" library_urn="urn:adsk.eagle:library:334" deviceset="R-US_" device="R0603" package3d_urn="urn:adsk.eagle:package:23555/2" value="220"/>
+<part name="R10" library="rcl" library_urn="urn:adsk.eagle:library:334" deviceset="R-US_" device="R0603" package3d_urn="urn:adsk.eagle:package:23555/2" value="4k7"/>
+<part name="R20" library="rcl" library_urn="urn:adsk.eagle:library:334" deviceset="R-US_" device="R0603" package3d_urn="urn:adsk.eagle:package:23555/2" value="4k7"/>
 <part name="+3V11" library="supply1" library_urn="urn:adsk.eagle:library:371" deviceset="+3V3" device=""/>
 <part name="GND24" library="supply1" library_urn="urn:adsk.eagle:library:371" deviceset="GND" device=""/>
-<part name="R21" library="rcl" library_urn="urn:adsk.eagle:library:334" deviceset="R-US_" device="R0603" package3d_urn="urn:adsk.eagle:package:23555/2" value="220"/>
+<part name="R21" library="rcl" library_urn="urn:adsk.eagle:library:334" deviceset="R-US_" device="R0603" package3d_urn="urn:adsk.eagle:package:23555/2" value="100"/>
 <part name="R22" library="rcl" library_urn="urn:adsk.eagle:library:334" deviceset="R-US_" device="R0603" package3d_urn="urn:adsk.eagle:package:23555/2" value="220"/>
 <part name="LED6" library="led" library_urn="urn:adsk.eagle:library:259" deviceset="LED" device="SML0603" package3d_urn="urn:adsk.eagle:package:15832/1"/>
 <part name="GND25" library="supply1" library_urn="urn:adsk.eagle:library:371" deviceset="GND" device=""/>
-<part name="R23" library="rcl" library_urn="urn:adsk.eagle:library:334" deviceset="R-US_" device="R0603" package3d_urn="urn:adsk.eagle:package:23555/2" value="220"/>
+<part name="R23" library="rcl" library_urn="urn:adsk.eagle:library:334" deviceset="R-US_" device="R0603" package3d_urn="urn:adsk.eagle:package:23555/2" value="10k"/>
 <part name="GND26" library="supply1" library_urn="urn:adsk.eagle:library:371" deviceset="GND" device=""/>
 <part name="GND27" library="supply1" library_urn="urn:adsk.eagle:library:371" deviceset="GND" device=""/>
@@
 <part name="C25" library="rcl" library_urn="urn:adsk.eagle:library:334" deviceset="C-EU" device="C0603" package3d_urn="urn:adsk.eagle:package:23616/2"/>
 <part name="GND28" library="supply1" library_urn="urn:adsk.eagle:library:371" deviceset="GND" device=""/>
-<part name="R24" library="rcl" library_urn="urn:adsk.eagle:library:334" deviceset="R-US_" device="R0603" package3d_urn="urn:adsk.eagle:package:23555/2" value="220"/>
-<part name="R25" library="rcl" library_urn="urn:adsk.eagle:library:334" deviceset="R-US_" device="R0603" package3d_urn="urn:adsk.eagle:package:23555/2" value="220"/>
-<part name="R26" library="rcl" library_urn="urn:adsk.eagle:library:334" deviceset="R-US_" device="R0603" package3d_urn="urn:adsk.eagle:package:23555/2" value="220"/>
-<part name="R27" library="rcl" library_urn="urn:adsk.eagle:library:334" deviceset="R-US_" device="R0603" package3d_urn="urn:adsk.eagle:package:23555/2" value="220"/>
+<part name="R24" library="rcl" library_urn="urn:adsk.eagle:library:334" deviceset="R-US_" device="R0603" package3d_urn="urn:adsk.eagle:package:23555/2" value="22"/>
+<part name="R25" library="rcl" library_urn="urn:adsk.eagle:library:334" deviceset="R-US_" device="R0603" package3d_urn="urn:adsk.eagle:package:23555/2" value="222"/>
+<part name="R26" library="rcl" library_urn="urn:adsk.eagle:library:334" deviceset="R-US_" device="R0603" package3d_urn="urn:adsk.eagle:package:23555/2" value="100k"/>
+<part name="R27" library="rcl" library_urn="urn:adsk.eagle:library:334" deviceset="R-US_" device="R0603" package3d_urn="urn:adsk.eagle:package:23555/2" value="1k5"/>
 <part name="+3V12" library="supply1" library_urn="urn:adsk.eagle:library:371" deviceset="+3V3" device=""/>
 <part name="USB3" library="microusb" deviceset="MICRO-USB" device=""/>

Commit message: initial commit add a backup file
Parts:
- removed IC3: CP2102, silabs:CP2102
- removed JP8: (no value), jumper:JP1Q
- removed LED2, LED3, LED4, LED5: (no value), led:LEDSML0603
- removed R16, R17, R18, R19: 220, rcl:R-US_R0603
- added C26, C27: (no value), rcl:C-EUC0603
- added IC7: (no value), usblc6:USBLC6-2SC6
- added IC8: CP2101, silabs-2:CP2101
- added JP9: JUMPER-3SMD, SparkFun:JUMPER-3SMD
- JP2: device jumper:JP3Q -> jumper:JP1Q
- JP6: value FIDUCIAL1X2 -> JUMPER-3SMD; device SparkFun:FIDUCIAL1X2 -> SparkFun:JUMPER-3SMD
Connections:
- net USB_DM renamed DW_N
- net USB_DP renamed DW_P
- removed net N$24: LED3.A, R17.2
- removed net N$25: LED4.A, R18.2
- removed net N$26: LED5.A, R19.2
- new net N$18: IC7.I/O1, R24.2
- net +3V3: now also C26.2, C27.2, JP2.1; no longer JP3.1
- net +5V: now also IC7.VBUS, IC8.REGIN, IC8.VBUS; no longer IC3.REGIN, IC3.VBUS
- net AN5: now also JP6.2; no longer JP2.4
- net AN6: now also JP9.2; no longer JP2.3
- net F3SWCLK: now also JP3.1; no longer JP8.1
- net F3SWDIO: now also JP3.2; no longer JP8.2
- net GND: now also C26.1, C27.1, IC7.GND, IC8.GND, IC8.GND@EXP, IC8.GND@M; no longer IC3.GND, IC3.GND@EXP, IC3.GND@M, LED2.C, LED3.C, LED4.C, LED5.C
- net N$16: now also IC8.!RST; no longer IC3.!RST
- net N$17: now also IC8.!SUSPEND; no longer IC3.!SUSPEND
- net N$19: now also IC8.TXD; no longer IC3.TXD
- net N$20: now also IC8.RXD; no longer IC3.RXD
- net N$21: now also IC7.I/O2, R25.2; no longer R24.2, USB3.D-
- net N$23: now also IC7.I/O_1, USB3.D-; no longer LED2.A, R16.2
- net N$40: now also IC7.I/O_2; no longer R25.2
- net N$5: now also IC8.VDD; no longer IC3.VDD
- net PA3: no longer R16.1
- net PA4: no longer R17.1
- net PA5: no longer R18.1
- net PA6: no longer R19.1
- net PC0: now also JP9.1; no longer JP2.5
- net PC1: now also JP6.1; no longer JP2.6
- net SCL: now also JP9.3; no longer JP2.1
- net SDA: now also JP6.3; no longer JP2.2
- net USB_N: now also IC8.D-; no longer IC3.D-
- net USB_P: now also IC8.D+; no longer IC3.D+
- net VDDA_PIN: now also JP2.2; no longer JP3.2
Other:
- note removed: "LED"
- moved on the sheet: C25, JP3, JP7, R24, R25, R26, R27, USB3

Commit message: initial commit, mainboard V2
Parts:
- added U$1: LOGO_PME2, Custom:LOGO_PME2
Connections:
- net BOOT0: now also JP1.4; no longer JP1.3
- net BOOT1: now also JP1.3; no longer JP1.4
- net N$1: now also JP1.5; no longer JP1.2
- net N$3: now also JP1.6; no longer JP1.1
- net N$33: now also JP1.1; no longer JP1.6
- net N$34: now also JP1.2; no longer JP1.5
Other:
- moved on the sheet: JP1
